Commit message: Fix launch file

File: ros2_ws/src/bur_gz/urdf/bur.urdf (robot description, URDF)
Before this commit: robot bur, 2 links, 1 joints
Links:
- added link bur/thruster2, mass 0.07; collision cylinder length=0.035 radius=0.05; visual cylinder length=0.035 radius=0.05
- added link bur/thruster3, mass 0.07; collision cylinder length=0.035 radius=0.05; visual cylinder length=0.035 radius=0.05
- added link bur/thruster4, mass 0.07; collision cylinder length=0.035 radius=0.05; visual cylinder length=0.035 radius=0.05
- added link bur/thruster5, mass 0.07; collision cylinder length=0.035 radius=0.05; visual cylinder length=0.035 radius=0.05
- added link bur/thruster6, mass 0.07; collision cylinder length=0.035 radius=0.05; visual cylinder length=0.035 radius=0.05
- added link bur/thruster7, mass 0.07; collision cylinder length=0.035 radius=0.05; visual cylinder length=0.035 radius=0.05
- added link bur/thruster8, mass 0.07; collision cylinder length=0.035 radius=0.05; visual cylinder length=0.035 radius=0.05
- link bur/base_link: geometry collision box size=0.25029927476882613 0.5005985495376523 0.12514963738441306; visual box size=0.25029927476882613 0.5005985495376523 0.12514963738441306
Joints:
- added joint thruster2: type fixed, parent bur/base_link, child bur/thruster2, origin xyz=0.1555 0.15 -0.0725 rpy=0 0 0.7853981634, axis 1 0 0
- added joint thruster3: type fixed, parent bur/base_link, child bur/thruster3, origin xyz=-0.1555 -0.15 -0.0725 rpy=0 0 0.7853981634, axis 1 0 0
- added joint thruster4: type fixed, parent bur/base_link, child bur/thruster4, origin xyz=-0.1555 0.15 -0.0725 rpy=0 0 0.7853981634, axis 1 0 0
- added joint thruster5: type fixed, parent bur/base_link, child bur/thruster5, origin xyz=0.13333333333333333 -0.26666666666666666 0 rpy=-0.7853981633974483 1.5707963267948966 0, axis 1 0 0
- added joint thruster6: type fixed, parent bur/base_link, child bur/thruster6, origin xyz=0.13333333333333333 0.26666666666666666 0 rpy=0.7853981633974483 1.5707963267948966 0, axis 1 0 0
- added joint thruster7: type fixed, parent bur/base_link, child bur/thruster7, origin xyz=-0.13333333333333333 -0.26666666666666666 0 rpy=0.7853981633974483 1.5707963267948966 0, axis 1 0 0
- added joint thruster8: type fixed, parent bur/base_link, child bur/thruster8, origin xyz=-0.13333333333333333 0.26666666666666666 0 rpy=-0.7853981633974483 1.5707963267948966 0, axis 1 0 0
- joint thruster1: origin xyz=0.1355 -0.1 -0.0725 rpy=0 0 0.7853981634 -> xyz=0.1555 -0.15 -0.0725 rpy=0 0 0.7853981634; type continuous -> fixed

File: ros2_ws/src/bur_gz/urdf/thruster.urdf.xacro (robot description, xacro)
@@ -36,5 +36,5 @@
       <xacro:insert_block name="origin" />
       <axis xyz="1 0 0" />
-      <parent link="${ns}/base_link">
+      <parent link="${ns}/base_link" />
       <child link="${ns}/thruster${thruster_id}" />
       <limits effort="-1" velocity="-1"/>

Commit message: Fix axes + add thruster stl files

File: ros2_ws/src/bur_gz/urdf/bur.urdf (robot description, URDF)
Before this commit: robot bur, 9 links, 8 joints
Links:
- added link bur/dlink
- link bur/thruster1: geometry collision mesh filename=file:///bur/ros2_ws/install/bur_gz/share/bur_gz/meshes/Impe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 scale=0.0007 0.0007 0.0007; visual mesh filename=file:///bur/ros2_ws/install/bur_gz/share/bur_gz/meshes/Impe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 scale=0.0007 0.0007 0.0007
- link bur/thruster2: geometry collision mesh filename=file:///bur/ros2_ws/install/bur_gz/share/bur_gz/meshes/Impe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 scale=0.0007 0.0007 0.0007; visual mesh filename=file:///bur/ros2_ws/install/bur_gz/share/bur_gz/meshes/Impe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 scale=0.0007 0.0007 0.0007
- link bur/thruster3: geometry collision mesh filename=file:///bur/ros2_ws/install/bur_gz/share/bur_gz/meshes/Impe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 scale=0.0007 0.0007 0.0007; visual mesh filename=file:///bur/ros2_ws/install/bur_gz/share/bur_gz/meshes/Impe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 scale=0.0007 0.0007 0.0007
- link bur/thruster4: geometry collision mesh filename=file:///bur/ros2_ws/install/bur_gz/share/bur_gz/meshes/Impe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 scale=0.0007 0.0007 0.0007; visual mesh filename=file:///bur/ros2_ws/install/bur_gz/share/bur_gz/meshes/Impe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 scale=0.0007 0.0007 0.0007
- link bur/thruster5: geometry collision mesh filename=file:///bur/ros2_ws/install/bur_gz/share/bur_gz/meshes/Impe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 scale=0.0007 0.0007 0.0007; visual mesh filename=file:///bur/ros2_ws/install/bur_gz/share/bur_gz/meshes/Impe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 scale=0.0007 0.0007 0.0007
- link bur/thruster6: geometry collision mesh filename=file:///bur/ros2_ws/install/bur_gz/share/bur_gz/meshes/Impe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 scale=0.0007 0.0007 0.0007; visual mesh filename=file:///bur/ros2_ws/install/bur_gz/share/bur_gz/meshes/Impe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 scale=0.0007 0.0007 0.0007
- link bur/thruster7: geometry collision mesh filename=file:///bur/ros2_ws/install/bur_gz/share/bur_gz/meshes/Impe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 scale=0.0007 0.0007 0.0007; visual mesh filename=file:///bur/ros2_ws/install/bur_gz/share/bur_gz/meshes/Impe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 scale=0.0007 0.0007 0.0007
- link bur/thruster8: geometry collision mesh filename=file:///bur/ros2_ws/install/bur_gz/share/bur_gz/meshes/Impe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 scale=0.0007 0.0007 0.0007; visual mesh filename=file:///bur/ros2_ws/install/bur_gz/share/bur_gz/meshes/Impe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 scale=0.0007 0.0007 0.0007
Joints:
- added joint bur/dummy_link: type fixed, parent bur/dlink, child bur/base_link, origin xyz=0 0 0 rpy=0 0 0
- joint thruster1: axis 1 0 0 -> 0 0 1; origin xyz=0.1555 -0.15 -0.0725 rpy=0 0 0.7853981634 -> xyz=0.1555 -0.15 -0.0725 rpy=0 0 0; type fixed -> continuous
- joint thruster2: axis 1 0 0 -> 0 0 1; origin xyz=0.1555 0.15 -0.0725 rpy=0 0 0.7853981634 -> xyz=0.1555 0.15 -0.0725 rpy=0 0 0; type fixed -> continuous
- joint thruster3: axis 1 0 0 -> 0 0 1; origin xyz=-0.1555 -0.15 -0.0725 rpy=0 0 0.7853981634 -> xyz=-0.1555 -0.15 -0.0725 rpy=0 0 0; type fixed -> continuous
- joint thruster4: axis 1 0 0 -> 0 0 1; origin xyz=-0.1555 0.15 -0.0725 rpy=0 0 0.7853981634 -> xyz=-0.1555 0.15 -0.0725 rpy=0 0 0; type fixed -> continuous
- joint thruster5: axis 1 0 0 -> 0 0 1; type fixed -> continuous
- joint thruster6: axis 1 0 0 -> 0 0 1; type fixed -> continuous
- joint thruster7: axis 1 0 0 -> 0 0 1; origin xyz=-0.13333333333333333 -0.26666666666666666 0 rpy=0.7853981633974483 1.5707963267948966 0 -> xyz=-0.13333333333333333 -0.26666666666666666 0 rpy=-0.7853981633974483 -1.5707963267948966 0; type fixed -> continuous
- joint thruster8: axis 1 0 0 -> 0 0 1; origin xyz=-0.13333333333333333 0.26666666666666666 0 rpy=-0.7853981633974483 1.5707963267948966 0 -> xyz=-0.13333333333333333 0.26666666666666666 0 rpy=0.7853981633974483 -1.5707963267948966 0; type fixed -> continuous

File: ros2_ws/src/bur_gz/urdf/bur.urdf.xacro (robot description, xacro)
@@ -67,14 +67,14 @@
   <xacro:include filename="thruster.urdf.xacro"/>
   <xacro:thruster thruster_id="1">
-    <origin xyz="0.1555 -0.15 -0.0725" rpy="0 0 0.7853981634"/>
+    <origin xyz="0.1555 -0.15 -0.0725" rpy="0 0 0"/>
   </xacro:thruster>
   <xacro:thruster thruster_id="2">
-    <origin xyz="0.1555 0.15 -0.0725" rpy="0 0 0.7853981634"/>
+    <origin xyz="0.1555 0.15 -0.0725" rpy="0 0 0"/>
   </xacro:thruster>
   <xacro:thruster thruster_id="3">
-    <origin xyz="-0.1555 -0.15 -0.0725" rpy="0 0 0.7853981634"/>
+    <origin xyz="-0.1555 -0.15 -0.0725" rpy="0 0 0"/>
   </xacro:thruster>
   <xacro:thruster thruster_id="4">
-    <origin xyz="-0.1555 0.15 -0.0725" rpy="0 0 0.7853981634"/>
+    <origin xyz="-0.1555 0.15 -0.0725" rpy="0 0 0"/>
   </xacro:thruster>
   <xacro:thruster thruster_id="5">
@@ -85,8 +85,8 @@
   </xacro:thruster>
   <xacro:thruster thruster_id="7">
-    <origin xyz="${-x_size / 3} ${-y_size / 3} 0" rpy="${pi/4} ${pi/2} 0"/>
+    <origin xyz="${-x_size / 3} ${-y_size / 3} 0" rpy="${-pi/4} ${-pi/2} 0"/>
   </xacro:thruster>
   <xacro:thruster thruster_id="8">
-    <origin xyz="${-x_size / 3} ${y_size / 3} 0" rpy="${-pi/4} ${pi/2} 0"/>
+    <origin xyz="${-x_size / 3} ${y_size / 3} 0" rpy="${pi/4} ${-pi/2} 0"/>
   </xacro:thruster>
   <xacro:if value="$(arg simulation)">

File: ros2_ws/src/bur_gz/urdf/thruster.urdf.xacro (robot description, xacro)
@@ -7,6 +7,8 @@
     <link name="${ns}/thruster${thruster_id}">
       <visual>
+        <origin xyz="0.10 0.10 0" rpy="${pi/2} ${pi} 0"/>
         <geometry>
-          <cylinder length="${prop_l}" radius="${prop_r}"/>
+          <!-- cylinder length="${prop_l}" radius="${prop_r}"/ -->
+          <mesh filename="file://$(find bur_gz)/meshes/Impeller.STL" scale="0.0007 0.0007 0.0007"/>
         </geometry>
         <xacro:if value="${thruster_id in [1,2,3,4]}">
@@ -18,7 +20,8 @@
       </visual>
       <collision>
-        <origin rpy="0 ${pi/2} 0"/>
+        <origin xyz="0.10 0.10 0" rpy="${pi/2} ${pi} 0"/>
         <geometry>
-          <cylinder length="${prop_l}" radius="${prop_r}"/>
+          <!-- cylinder length="${prop_l}" radius="${prop_r}"/ -->
+          <mesh filename="file://$(find bur_gz)/meshes/Impeller.STL" scale="0.0007 0.0007 0.0007"/>
         </geometry>
       </collision>
@@ -34,5 +37,5 @@
     <joint name="thruster${thruster_id}" type="continuous">
       <xacro:insert_block name="origin" />
-      <axis xyz="1 0 0" />
+      <axis xyz="0 0 1" />
       <parent link="${ns}/base_link" />
       <child link="${ns}/thruster${thruster_id}" />
