Commit message: Create basic model for robot

File: ros2_ws/src/bur_gz/urdf/bur.urdf.xacro (robot description, xacro)
@@ -1,3 +1,3 @@
-<?xml version="1.0">
+<?xml version="1.0"?>
 <robot xmlns:xacro="http://www.ros.org/wiki/xacro" name="bur">
   <!-- Arguments -->
@@ -8,8 +8,79 @@
   <xacro:property name="density" value="$(arg density)"/>
   <!-- Import modules -->
-  <xacro:include filename="thrusters.xacro"/>
+  <xacro:include filename="helpers.urdf.xacro"/>
+  <xacro:include filename="colors.urdf.xacro"/>
+  <xacro:include filename="thruster.urdf.xacro"/>
   <!-- Dimensions -->
   <xacro:property name="x_size" value="0.40"/>
   <xacro:property name="y_size" value="0.80"/>
-  <xacro:property name="z_size" value="0.40"/>
+  <xacro:property name="z_size" value="0.20"/>
+  <xacro:property name="mass" value="14.8"/>
+  <xacro:property name="prop_mass" value="0.07"/>
+  <xacro:property name="prop_mass" value="0.07"/>
+  <!-- to set correct buoyancy volume with 1 % positive factor -->
+  <xacro:property name="buoyant_correction" value="${1.01*pow((mass + 6*prop_mass)/(density*x_size*y_size*z_size), 1./3)}"/>
+  <!-- Center of buoyancy -->
+  <xacro:property name="z_cob" value="${-buoyant_correction*z_size/4}"/>
+  <!-- Center of gravity -->
+  <xacro:property name="z_cog" value="${-buoyant_correction*z_size}"/>
+  <!-- link name="${ns}/base_link" -->
+  <link name="base_link">
+    <inertial>
+      <mass value="${mass}"/>
+      <origin xyz="0 0 ${z_cog}"/>
+      <!-- BlueROV2 values from "Model Predictive Control for the BlueROV2",
+           Emil Már Einarsson, Andris Lipenitis, Master thesis, 2020
+           for now make Ignition crash?-->
+      <!--         <inertia ixx="0.21" ixy="0.00" ixz="0.00" iyy="0.245" iyz="0.00" izz="0.245"/> -->
+      <inertia ixx="5.2539" ixy="0.0144" ixz="0.3341" iyy="7.9420" iyz="0.026" izz="6.9123"/>
+      <!-- Perfect rectangle -->
+      <!--        <inertia
+           ixx="${mass/12*(y_size*y_size+z_size*z_size)}" ixy="0.0" ixz="0.0"
+           iyy="${mass/12*(x_size*x_size + z_size*z_size)}" iyz="0.0"
+           izz="${mass/12*(x_size*x_size + y_size*y_size)}" />-->
+    </inertial>
+    <visual>
+      <geometry>
+        <box size="${x_size*buoyant_correction} ${y_size*buoyant_correction} ${z_size*buoyant_correction}"/>
+      </geometry>
+      <material name="grey"/>
+    </visual>
+    <collision>
+      <origin xyz="0 0 ${z_cob}"/>
+      <!-- Box adjusted for buoyancy -->
+      <geometry>
+        <box size="${x_size*buoyant_correction} ${y_size*buoyant_correction} ${z_size*buoyant_correction}"/>
+      </geometry>
+    </collision>
+    <!--    <gazebo>
+         <velocity_decay>
+         <linear>-250.15 -70.364 -170.955</linear>
+         <angular>1.888 0.761 3.744</angular>
+         </velocity_decay>
+         </gazebo>-->
+  </link>
+  <xacro:thruster thruster_id="1">
+    <origin xyz="0.1555 -0.15 -0.0725" rpy="0 0 0.7853981634"/>
+  </xacro:thruster>
+  <xacro:thruster thruster_id="2">
+    <origin xyz="0.1555 0.15 -0.0725" rpy="0 0 0.7853981634"/>
+  </xacro:thruster>
+  <xacro:thruster thruster_id="3">
+    <origin xyz="-0.1555 -0.15 -0.0725" rpy="0 0 0.7853981634"/>
+  </xacro:thruster>
+  <xacro:thruster thruster_id="4">
+    <origin xyz="-0.1555 0.15 -0.0725" rpy="0 0 0.7853981634"/>
+  </xacro:thruster>
+  <xacro:thruster thruster_id="5">
+    <origin xyz="${x_size / 3} ${-y_size / 3} 0" rpy="${-pi/4} ${pi/2} 0"/>
+  </xacro:thruster>
+  <xacro:thruster thruster_id="6">
+    <origin xyz="${x_size / 3} ${y_size / 3} 0" rpy="${pi/4} ${pi/2} 0"/>
+  </xacro:thruster>
+  <xacro:thruster thruster_id="7">
+    <origin xyz="${-x_size / 3} ${-y_size / 3} 0" rpy="${pi/4} ${pi/2} 0"/>
+  </xacro:thruster>
+  <xacro:thruster thruster_id="8">
+    <origin xyz="${-x_size / 3} ${y_size / 3} 0" rpy="${-pi/4} ${pi/2} 0"/>
+  </xacro:thruster>
 </robot>

File: ros2_ws/src/bur_gz/urdf/helpers.urdf.xacro (robot description, xacro)
@@ -1,4 +1,5 @@
-<?xml version="1.0">
-<robot xmlns:xacro="http://www.ros.org/wiki/xacro" name="bur">
+<?xml version="1.0"?>
+<robot xmlns:xacro="http://www.ros.org/wiki/xacro">
+  <!-- Helper methods -->
   <xacro:macro name="gen_box" params="name x y z">
     <link name="${name}">

File: ros2_ws/src/bur_gz/urdf/thruster.urdf.xacro (robot description, xacro)
@@ -1,18 +1,22 @@
-<?xml version="1.0">
-<robot xmlns:xacro="http://www.ros.org/wiki/xacro" name="bur">
+<?xml version="1.0"?>
+<robot xmlns:xacro="http://www.ros.org/wiki/xacro">
+  <!-- Properties -->
+  <xacro:property name="prop_r" value="0.05"/>
+  <xacro:property name="prop_l" value="0.035"/>
   <xacro:macro name="thruster" params="thruster_id *origin">
     <link name="${ns}/thruster${thruster_id}">
     <visual>
       <geometry>
-        <xacro:if value="${thruster_id in [1,2,5]}">
-          <mesh filename="${prop_mesh_cw}"/>
-        </xacro:if>
-        <xacro:unless value="${thruster_id in [1,2,5]}">
-          <mesh filename="${prop_mesh_ccw}"/>
-        </xacro:unless>
+        <cylinder length="${prop_l}" radius="${prop_r}"/>
       </geometry>
+      <xacro:if value="${thruster_id in [1,2,3,4]}">
+        <material name="yellow"/>
+      </xacro:if>
+      <xacro:if value="${thruster_id in [5,6,7,8]}">
+        <material name="red"/>
+      </xacro:if>
     </visual>
     <collision>
-      <origin rpy="0 ${PI/2} 0"/>
+      <origin rpy="0 ${pi/2} 0"/>
       <geometry>
         <cylinder length="${prop_l}" radius="${prop_r}"/>
@@ -31,11 +35,7 @@
     <joint name="thruster${thruster_id}" type="continuous">
       <xacro:insert_block name="origin" />
-      <xacro:if value="${thruster_id in [1,2,5]}">
-        <axis xyz="1 0 0" />
-      </xacro:if>
-      <xacro:unless value="${thruster_id in [1,2,5]}">
-        <axis xyz="-1 0 0" />
-      </xacro:unless>
-      <parent link="${ns}/base_link" />
+      <axis xyz="1 0 0" />
+      <!-- parent link="${ns}/base_link" /-->
+      <parent link="base_link" />
       <child link="${ns}/thruster${thruster_id}" />
       <limits effort="-1" velocity="-1"/>

Commit message: Commit what I have

File: ros2_ws/src/bur_gz/urdf/bur.urdf.xacro (robot description, xacro)
@@ -24,6 +24,5 @@
   <!-- Center of gravity -->
   <xacro:property name="z_cog" value="${-buoyant_correction*z_size}"/>
-  <!-- link name="${ns}/base_link" -->
-  <link name="base_link">
+  <link name="${ns}/base_link">
     <inertial>
       <mass value="${mass}"/>

File: ros2_ws/src/bur_gz/urdf/thruster.urdf.xacro (robot description, xacro)
@@ -33,9 +33,8 @@
     </link>
     <!-- Joint between thruster link and vehicle base link -->
-    <joint name="thruster${thruster_id}" type="continuous">
+    <joint name="thruster${thruster_id}" type="fixed">
       <xacro:insert_block name="origin" />
       <axis xyz="1 0 0" />
-      <!-- parent link="${ns}/base_link" /-->
-      <parent link="base_link" />
+      <parent link="${ns}/base_link">
       <child link="${ns}/thruster${thruster_id}" />
       <limits effort="-1" velocity="-1"/>

Commit message: Make gazebo sim (still not working)

File: ros2_ws/src/bur_gz/urdf/bur.urdf.xacro (robot description, xacro)
@@ -7,8 +7,4 @@
   <xacro:property name="ns" value="$(arg namespace)"/>
   <xacro:property name="density" value="$(arg density)"/>
-  <!-- Import modules -->
-  <xacro:include filename="helpers.urdf.xacro"/>
-  <xacro:include filename="colors.urdf.xacro"/>
-  <xacro:include filename="thruster.urdf.xacro"/>
   <!-- Dimensions -->
   <xacro:property name="x_size" value="0.40"/>
@@ -59,4 +55,9 @@
          </gazebo>-->
   </link>
+  <!-- Import modules -->
+  <xacro:include filename="helpers.urdf.xacro"/>
+  <xacro:include filename="colors.urdf.xacro"/>
+  <xacro:include filename="hydrodynamics.urdf.xacro"/>
+  <xacro:include filename="thruster.urdf.xacro"/>
   <xacro:thruster thruster_id="1">
     <origin xyz="0.1555 -0.15 -0.0725" rpy="0 0 0.7853981634"/>
@@ -83,3 +84,24 @@
     <origin xyz="${-x_size / 3} ${y_size / 3} 0" rpy="${-pi/4} ${pi/2} 0"/>
   </xacro:thruster>
+  <xacro:if value="$(arg simulation)">
+    <gazebo>
+      <plugin filename="ignition-gazebo-joint-state-publisher-system" name="ignition::gazebo::systems::JointStatePublisher"/>
+      <plugin
+          filename="ignition-gazebo-odometry-publisher-system"
+          name="ignition::gazebo::systems::OdometryPublisher">
+        <odom_frame>${ns}/odom</odom_frame>
+        <dimensions>3</dimensions>
+        <robot_base_frame>${ns}/base_link</robot_base_frame>
+        <odom_publish_frequency>10</odom_publish_frequency>
+      </plugin>
+      <plugin
+          filename="ignition-gazebo-pose-publisher-system"
+          name="ignition::gazebo::systems::PosePublisher">
+        <publish_link_pose>false</publish_link_pose>
+        <publish_collision_pose>false</publish_collision_pose>
+        <publish_visual_pose>false</publish_visual_pose>
+        <publish_nested_model_pose>true</publish_nested_model_pose>
+      </plugin>
+    </gazebo>
+  </xacro:if>
 </robot>

File: ros2_ws/src/bur_gz/urdf/thruster.urdf.xacro (robot description, xacro)
@@ -6,29 +6,28 @@
   <xacro:macro name="thruster" params="thruster_id *origin">
     <link name="${ns}/thruster${thruster_id}">
-    <visual>
-      <geometry>
-        <cylinder length="${prop_l}" radius="${prop_r}"/>
-      </geometry>
-      <xacro:if value="${thruster_id in [1,2,3,4]}">
-        <material name="yellow"/>
-      </xacro:if>
-      <xacro:if value="${thruster_id in [5,6,7,8]}">
-        <material name="red"/>
-      </xacro:if>
-    </visual>
-    <collision>
-      <origin rpy="0 ${pi/2} 0"/>
-      <geometry>
-        <cylinder length="${prop_l}" radius="${prop_r}"/>
-      </geometry>
-    </collision>
-    <inertial>
-      <!-- thruster axis is X -->
-      <origin xyz="${prop_l/2} 0 0" rpy="0 0 0" />
-      <mass value="${prop_mass}" />
-      <inertia  izz="${prop_mass*prop_r*prop_r / 4  + prop_mass*prop_l*prop_l / 12}" ixy="0.0"  ixz="0.0"
-        iyy="${prop_mass*prop_r*prop_r / 4  + prop_mass*prop_l*prop_l / 12}" iyz="0.0"
-        ixx="${prop_mass*prop_r*prop_r / 2}" />
-    </inertial>
+      <visual>
+        <geometry>
+          <cylinder length="${prop_l}" radius="${prop_r}"/>
+        </geometry>
+        <xacro:if value="${thruster_id in [1,2,3,4]}">
+          <material name="yellow"/>
+        </xacro:if>
+        <xacro:if value="${thruster_id in [5,6,7,8]}">
+          <material name="red"/>
+        </xacro:if>
+      </visual>
+      <collision>
+        <origin rpy="0 ${pi/2} 0"/>
+        <geometry>
+          <cylinder length="${prop_l}" radius="${prop_r}"/>
+        </geometry>
+      </collision>
+      <inertial>
+        <!-- thruster axis is X -->
+        <origin xyz="${prop_l/2} 0 0" rpy="0 0 0" />
+        <mass value="${prop_mass}" />
+        <inertia  izz="${prop_mass*prop_r*prop_r / 4  + prop_mass*prop_l*prop_l / 12}" ixy="0.0"  ixz="0.0"
+                  iyy="${prop_mass*prop_r*prop_r / 4  + prop_mass*prop_l*prop_l / 12}" iyz="0.0" ixx="${prop_mass*prop_r*prop_r / 2}" />
+      </inertial>
     </link>
     <!-- Joint between thruster link and vehicle base link -->

Commit message: Fix thrusters

File: ros2_ws/src/bur_gz/urdf/bur.urdf.xacro (robot description, xacro)
@@ -20,4 +20,10 @@
   <!-- Center of gravity -->
   <xacro:property name="z_cog" value="${-buoyant_correction*z_size}"/>
+  <link name="${ns}/dlink" />
+  <joint name="${ns}/dummy_link" type="fixed">
+    <origin xyz="0 0 0" rpy="0 0 0" />
+    <parent link="${ns}/dlink" />
+    <child link="${ns}/base_link" />
+  </joint>
   <link name="${ns}/base_link">
     <inertial>
@@ -92,5 +98,5 @@
         <odom_frame>${ns}/odom</odom_frame>
         <dimensions>3</dimensions>
-        <robot_base_frame>${ns}/base_link</robot_base_frame>
+        <robot_base_frame>${ns}/dlink</robot_base_frame>
         <odom_publish_frequency>10</odom_publish_frequency>
       </plugin>

File: ros2_ws/src/bur_gz/urdf/helpers.urdf.xacro (robot description, xacro)
@@ -2,5 +2,5 @@
 <robot xmlns:xacro="http://www.ros.org/wiki/xacro">
   <!-- Helper methods -->
-  <xacro:macro name="gen_box" params="name x y z">
+  <xacro:macro name="box" params="name x y z">
     <link name="${name}">
       <visual>

File: ros2_ws/src/bur_gz/urdf/hydrodynamics.urdf.xacro (robot description, xacro)
@@ -3,5 +3,5 @@
   <gazebo>
     <plugin filename="ignition-gazebo-hydrodynamics-system" name="ignition::gazebo::systems::Hydrodynamics">
-      <link_name>${ns}/base_link</link_name>
+      <link_name>${ns}/dlink</link_name>
       <xDotU>-5.5</xDotU>
       <yDotV>-12.7</yDotV>

File: ros2_ws/src/bur_gz/urdf/thruster.urdf.xacro (robot description, xacro)
@@ -32,30 +32,29 @@
     </link>
     <!-- Joint between thruster link and vehicle base link -->
-    <joint name="thruster${thruster_id}" type="fixed">
+    <joint name="thruster${thruster_id}" type="continuous">
       <xacro:insert_block name="origin" />
       <axis xyz="1 0 0" />
       <parent link="${ns}/base_link" />
       <child link="${ns}/thruster${thruster_id}" />
-      <limits effort="-1" velocity="-1"/>
     </joint>
     <!-- ignition topic is /model/{ns}/joint/{joint_name}/cmd_pos -->
-    <!--    <xacro:if value="$(arg simulation)"> -->
-    <gazebo>
-      <plugin
-        filename="ignition-gazebo-thruster-system"
-        name="ignition::gazebo::systems::Thruster">
-        <namespace>${ns}</namespace>
-        <joint_name>thruster${thruster_id}</joint_name>
-        <topic>thruster${thruster_id}/cmd</topic>
-        <thrust_coefficient>0.011</thrust_coefficient>
-        <fluid_density>${density}</fluid_density>
-        <propeller_diameter>${2*prop_r}</propeller_diameter>
-        <velocity_control>true</velocity_control>
-        <use_angvel_cmd>false</use_angvel_cmd>
-        <max_thrust_cmd>40</max_thrust_cmd>
-        <min_thrust_cmd>-40</min_thrust_cmd>
-      </plugin>
-    </gazebo>
-    <!--  </xacro:if> -->
+    <xacro:if value="$(arg simulation)">
+      <gazebo>
+        <plugin
+            filename="ignition-gazebo-thruster-system"
+            name="ignition::gazebo::systems::Thruster">
+          <namespace>${ns}</namespace>
+          <joint_name>thruster${thruster_id}</joint_name>
+          <topic>thruster${thruster_id}/cmd</topic>
+          <thrust_coefficient>0.011</thrust_coefficient>
+          <fluid_density>${density}</fluid_density>
+          <propeller_diameter>${2*prop_r}</propeller_diameter>
+          <velocity_control>true</velocity_control>
+          <use_angvel_cmd>false</use_angvel_cmd>
+          <max_thrust_cmd>40</max_thrust_cmd>
+          <min_thrust_cmd>-40</min_thrust_cmd>
+        </plugin>
+      </gazebo>
+    </xacro:if>
   </xacro:macro>
 </robot>

Commit message: Unfuck IMU

File: ros2_ws/src/bur_gz/urdf/bur.urdf.xacro (robot description, xacro)
@@ -66,4 +66,5 @@
   <xacro:include filename="hydrodynamics.urdf.xacro"/>
   <xacro:include filename="thruster.urdf.xacro"/>
+  <xacro:include filename="imu.urdf.xacro"/>
   <xacro:thruster thruster_id="1">
     <origin xyz="0.1555 -0.15 -0.0725" rpy="0 0 0"/>

File: ros2_ws/src/bur_gz/urdf/imu.urdf.xacro (robot description, xacro)
@@ -2,22 +2,35 @@
 <robot xmlns:xacro="http://www.ros.org/wiki/xacro">
   <xacro:include filename="helpers.urdf.xacro"/>
-  <xacro:box name="${ns}/imu_link" x="0.5" y="0.5" z="0.5" />
+  <gazebo>
+    <plugin filename="gz-sim-imu-system"
+        name="gz::sim::systems::Imu">
+    </plugin>
+  </gazebo>
+  <link name="${ns}/imu_link">
+    <visual>
+      <geometry>
+        <box size="0.01 0.01 0.01" />
+      </geometry>
+      <material name="green" />
+    </visual>
+    <collision>
+      <geometry>
+        <box size="0.01 0.01 0.01" />
+      </geometry>
+    </collision>
+  </link>
   <joint name="imu_joint" type="fixed">
     <axis xyz="1 0 0"/> <!-- 0 1 0 -->
-    <origin xyz="0 0 0.19"/>
+    <origin xyz="0 0 0.06"/>
     <parent link="${ns}/base_link"/>
     <child link="${ns}/imu_link"/>
   </joint>
-  <gazebo>
-    <controller:gazebo_ros_imu name="imu_controller" plugin="libgazebo_ros_imu.so">
-      <alwaysOn>true</alwaysOn>
-      <updateRate>50.0</updateRate>
-      <bodyName>${ns}/imu_link</bodyName>
-      <topicName>${ns}/imu_data</topicName>
-      <gaussianNoise>2.89e-08</gaussianNoise>
-      <xyzOffsets>0 0 0</xyzOffsets>
-      <rpyOffsets>0 0 0</rpyOffsets>
-      <interface:position name="imu_position"/>
-    </controller:gazebo_ros_imu>
+  <gazebo reference="${ns}/imu_link">
+    <sensor name="imu_sensor" type="imu">
+      <always_on>1</always_on>
+      <update_rate>1</update_rate>
+      <visualize>true</visualize>
+      <topic>imu</topic>
+    </sensor>
   </gazebo>
 </robot>

Commit message: Commit what I have
Signed-off-by: Prabhvir Babra <theprabab@gmail.com>

File: ros2_ws/src/bur_gz/urdf/bur.urdf.xacro (robot description, xacro)
@@ -67,4 +67,5 @@
   <xacro:include filename="thruster.urdf.xacro"/>
   <xacro:include filename="imu.urdf.xacro"/>
+  <xacro:include filename="camera.urdf.xacro"/>
   <xacro:thruster thruster_id="1">
     <origin xyz="0.1555 -0.15 -0.0725" rpy="0 0 0"/>
@@ -91,4 +92,7 @@
     <origin xyz="${-x_size / 3} ${y_size / 3} 0" rpy="${pi/4} ${-pi/2} 0"/>
   </xacro:thruster>
+  <xacro:camera camera_id="1">
+    <origin xyz="0.1 0 0.06" rpy="0 0 0" />
+  </xacro:camera>
   <xacro:if value="$(arg simulation)">
     <gazebo>
